File: b241/LET/project/hw/LET-project.kicad_sch (KiCad schematic)
At the start: 0 parts

Commit message: let project
Parts:
- added C1: 10uF, symbol Device:C
- added C10, C9: TBD, symbol Device:C
- added C11, C12: C, symbol Device:C
- added C2, C7: 1uF, symbol Device:C
- added C3, C4, C5, C6: 100nF, symbol Device:C
- added C8: 10nF, symbol Device:C
- added D1: SS14, Diode_SMD:D_SMA, symbol Diode:SS14
- added J1: USB_C_Receptacle_USB2.0_14P, symbol Connector:USB_C_Receptacle_USB2.0_14P
- added L1: 2nH, symbol Device:L
- added L2: 24nH, symbol Device:L
- added R1, R2: 5k1, symbol Device:R
- added U1: ESP32-C6, Package_DFN_QFN:QFN-40-1EP_5x5mm_P0.4mm_EP3.6x3.6mm, symbol PCM_Espressif:ESP32-C6
- added U2: USBLC6-2P6, Package_TO_SOT_SMD:SOT-666, symbol Power_Protection:USBLC6-2P6
- added Y1: ABM11W-40.0000MHZ-7-D1X-T3, ABM11W300000MHZ4B1UT3, symbol SamacSys Parts:ABM11W-40.0000MHZ-7-D1X-T3
- added Y2: ECS-.327-12.5-34B-C-TR, ECS32712534BCTR, symbol SamacSys Parts:ECS-.327-12.5-34B-C-TR
Connections:
- new net: J1.A6 (D+), J1.B6 (D+), U2.1 (I/O1)
- new net: J1.A7 (D-), J1.B7 (D-), U2.3 (I/O2)
- new net: C9.1, L2.2, Y1.1 (X1)
- new net: D1.2 (A), J1.A4 (VBUS), J1.A9 (VBUS), J1.B4 (VBUS), J1.B9 (VBUS)
- new net: J1.B5 (CC2), R1.1
- new net: J1.A5 (CC1), R2.1
- new net +3V3: C1.2, C2.2, C3.2, C5.1, C6.1, C7.1, C8.1, L1.1, U1.28 (VDDPST2), U1.37 (VDDA1), U1.40 (VDDA2), U1.5 (VDDPST1)
- new net +5V: D1.1 (K), U2.5 (VBUS)
- new net ANT: U1.1 (ANT)
- new net GND: C1.1, C10.2, C11.2, C12.2, C2.1, C3.1, C4.1, C5.2, C6.2, C7.2, C8.2, C9.2, J1.A1 (GND), J1.A12 (GND), J1.B1 (GND), J1.B12 (GND), J1.S1 (SHIELD), R1.2, R2.2, U1.41 (GND), U2.2 (GND), Y1.2 (GND_1), Y1.4 (GND_2)
- new net USB_D+: U1.19 (GPIO13/USB_D+), U2.6 (I/O1)
- new net USB_D-: U1.18 (GPIO12/USB_D-), U2.4 (I/O2)
- new net VDDA3P3: C4.2, L1.2, U1.2 (VDDA3P3), U1.3 (VDDA3P3)
- new net XTAL+: L2.1, U1.39 (XTAL_P)
- new net XTAL-: C10.1, U1.38 (XTAL_N), Y1.3 (X2)
- new net XTAL_32+: C11.1, U1.6 (GPIO0/XTAL_32K_P/ADC1_CH0), Y2.2 (OUT/IN)
- new net XTAL_32-: C12.1, U1.7 (GPIO1/XTAL_32K_N/ADC1_CH1), Y2.
Other:
- removed sheet SOC
- note added: "External Crystal Clock Source"
- note added: "RTC Clock Source"
- note added: "VDD coupling"
- note added: "VDDA coupling"
- note added: "VDDA3P3 coupling"
- company: (none) -> FEE CTU
- title: (none) -> Thread sensor

Commit message: finished schematic
Parts:
- removed D1: SS14, Diode_SMD:D_SMA, symbol Diode:SS14
- removed U2: USBLC6-2P6, Package_TO_SOT_SMD:SOT-666, symbol Power_Protection:USBLC6-2P6
- added AE1: Antenna_Chip, symbol Device:Antenna_Chip
- added C13, C14: TBD, symbol Device:C
- added C15, C16: 100nF, symbol Device:C
- added C17, C18, C19: 1uF, symbol Device:C
- added D1: ESD7002WTT1G, Package_TO_SOT_SMD:SOT-23-3, symbol Power_Protection:ESDA5V3L
- added D2, D3: MBRAF260T3G, SODFL5126X110N, symbol Device:D_Schottky
- added IC1: NCP187AMT330TAG, SON65P200X200X80-7N, symbol SamacSys Parts:NCP187AMT330TAG
- added J2, J4: Conn_01x03, symbol Connector_Generic:Conn_01x03
- added J3: Conn_01x02, symbol Connector_Generic:Conn_01x02
- added J5: Conn_01x04, symbol Connector_Generic:Conn_01x04
- added L3: TBD, symbol Device:L
- added Q1, Q3: Q_PMOS_DGS, symbol Device:Q_PMOS_DGS
- added Q2, Q4: Q_NMOS_DGS, symbol Device:Q_NMOS_DGS
- added R10: 10k, symbol Device:R
- added R11, R12: 4k7, symbol Device:R
- added R3, R4, R6, R7: TBD, symbol Device:R
- added R5, R9: 1k, symbol Device:R
- added R8: 100k, symbol Device:R
- added Z1: 1SMB5934BT3G, DIOM5436X247N, symbol Device:D_Zener
- renumbered C7 to C1, C8 to C10, C1 to C2, C2 to C3, C3 to C4, C4 to C5, C5 to C6, C6 to C7, C9 to C8, C10 to C9
Connections:
- net +3V3: now also C18.1, IC1.5 (SNS), IC1.6 (OUT), Q1.3 (S), Q3.3 (S), R10.2, R4.1, R7.1, R8.1
- net +5V: now also J1.A4 (VBUS), J1.A9 (VBUS), J1.B4 (VBUS), J1.B9 (VBUS), D3.2 (A), Z1.1 (K)
- net ANT: now also C13.1, L3.1
- net GND: now also AE1.1 (FEED), C13.2, C14.2, C15.2, C16.2, C17.2, C18.2, C19.2, D1.3 (A), IC1.3 (GND_1), IC1.7 (GND_2), J2.2 (Pin_2), J3.2 (Pin_2), J4.2 (Pin_2), J5.1 (Pin_1), Q2.3 (S), Q4.3 (S), R11.2, R12.2, R5.2, R9.2, Z1.2 (A)
- net USB_D+: now also J1.A6 (D+), J1.B6 (D+), D1.1 (K)
- net USB_D-: now also J1.A7 (D-), J1.B7 (D-), D1.2 (K)
- net ADC_IN1_EN: now reaches U1.14 (GPIO8)
- net ADC_IN1_EN: now also Q2.2 (G), R5.1
- net ADC_IN2_EN: now reaches U1.15 (GPIO9)
- net ADC_IN2_EN: now also Q4.2 (G), R9.1
- net SDA: now reaches U1.16 (GPIO10)
- net SDA: now also J5.3 (Pin_3), R11.1
- net SCL: now reaches U1.17 (GPIO11)
- net SCL: now also J5.2 (Pin_2), R12.1
- net CHIP_PU: now reaches U1.4 (CHIP_PU)
- net CHIP_PU: now also C19.1, R10.1
- net ADC_CH2: now reaches U1.8 (GPIO2/FSPIQ/ADC1_CH2)
- net ADC_CH2: now also C15.1, J2.1 (Pin_1)
- net ADC_CH3: now reaches U1.9 (GPIO3/ADC1_CH3)
- net ADC_CH3: now also C16.1, J4.1 (Pin_1)
- new net: J2.3 (Pin_3), Q1.1 (D)
- new net: D2.2 (A), J3.1 (Pin_1)
- new net: J4.3 (Pin_3), Q3.1 (D)
- new net: AE1.2 (PCB_Trace), C14.1, L3.2
- new net: Q1.2 (G), R3.1, R4.2
- new net: Q4.1 (D), R6.2
- new net: IC1.4 (PG), R8.2
- new net: Q3.2 (G), R6.1, R7.2
- new net: Q2.1 (D), R3.2
- new net +3.3V: J5.4 (Pin_4)
- new net 5V-merged: C17.1, D2.1 (K), D3.1 (K), IC1.1 (IN), IC1.2 (EN)
Other:
- note added: "Analog In 1"
- note added: "Analog In 2"
- note added: "CL = C8 * C9 / (C8 + C9) C8 = C9 CL = 7 pF"
- note added: "Chip power-up"
- note added: "I2C connection"
- note added: "MCU"
- note added: "RF matching"
- note added: "USB conn"
- note added: "power supply"
- company: FEE CTU -> (none)
- title: Thread sensor -> Thread enabled biosensor
- moved on the sheet: R2, U1

Commit message: LET project update
Parts:
- C1, C10, C11, C12, C13, C14, C15, C16, C17, C18, C19, C2, C3, C4, C5, C6, C7, C8, C9: footprint (none) -> Capacitor_SMD:C_0805_2012Metric
- D2, D3: footprint SODFL5126X110N -> SemacSys:SODFL5126X110N
- IC1: footprint SON65P200X200X80-7N -> SemacSys:SON65P200X200X80-7N
- L1, L2, L3: footprint (none) -> Inductor_SMD:L_0603_1608Metric
- R1, R2: footprint (none) -> RESC3225X60N; Height (none) -> 0.6; Manufacturer_Name (none) -> Vishay; Manufacturer_Part_Number (none) -> CRCW12105K10FKEA
- R10, R11, R12, R3, R4, R6, R7, R8: footprint (none) -> Resistor_SMD:R_0603_1608Metric
- R5, R9: footprint (none) -> RESC3225X60N; Height (none) -> 0.6; Manufacturer_Name (none) -> Vishay; Manufacturer_Part_Number (none) -> CRCW12101K00FKTA; Mouser Part Number (none) -> 71-CRCW1210-1.0K; Mouser Price/Stock (none) -> https://www.mouser.co.uk/ProductDetail/Vishay-Dale/CRCW1210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
